Commit message: Update

File: workspace/src/follower_scene/urdf/follower_robot.xacro (robot description, xacro)
@@ -76,5 +76,7 @@
             <mass value="0.001"/>
             <origin xyz="0 0 0" rpy="0 0 0"/>
-            <inertia ixx="1e-6" ixy="0" ixz="0" iyy="1e-6" iyz="0" izz="1e-6"/>
+            <inertia ixx="1e-6" ixy="0" ixz="0"
+                    iyy="1e-6" iyz="0"
+                    izz="1e-6"/>
         </inertial>
     </link>

File: workspace/src/follower_scene/urdf/leader_robot.xacro (robot description, xacro)
@@ -76,5 +76,7 @@
             <mass value="0.001"/>
             <origin xyz="0 0 0" rpy="0 0 0"/>
-            <inertia ixx="1e-6" ixy="0" ixz="0" iyy="1e-6" iyz="0" izz="1e-6"/>
+            <inertia ixx="1e-6" ixy="0" ixz="0"
+                    iyy="1e-6" iyz="0"
+                    izz="1e-6"/>
         </inertial>
     </link>
@@ -127,18 +129,16 @@
         <visual>
             <origin xyz="0 0 0" rpy="0 1.5708 0"/>
-            <geometry>
-                <box size="0.1 0.1 0.01"/>
-            </geometry>
+            <geometry><box size="0.1 0.1 0.01"/></geometry>
         </visual>
         <collision>
             <origin xyz="0 0 0" rpy="0 1.5708 0"/>
-            <geometry>
-                <box size="0.1 0.1 0.01"/>
-            </geometry>
+            <geometry><box size="0.1 0.1 0.01"/></geometry>
         </collision>
         <inertial>
             <mass value="0.05"/>
             <origin xyz="0 0 0" rpy="0 1.5708 0"/>
-            <inertia ixx="0.0001" ixy="0" ixz="0" iyy="0.0001" iyz="0" izz="0.0001"/>
+            <inertia ixx="0.0001" ixy="0" ixz="0"
+                    iyy="0.0001" iyz="0"
+                    izz="0.0001"/>
         </inertial>
     </link>
